File: esp32-nano.kicad_pcb (KiCad board)
At the start: 2 copper layers, 52.8 x 21.3 mm, 45 parts, among them K1 SW_MEC_5E, K2 SW_MEC_5E, P2 Conn_01x12, P3 Conn_01x18, U1 CP2102N-A01-GQFN28, U2 ME6211C33M5G, U3 MPU-6050, U4 ESP32PICO_D4, U5 OLED-12880

Commit message: .
Parts:
- turned R3 to 180 degrees
Routing:
- net Net-(K1-Pad3): track 0.00 -> 31.9 mm
- net GPIO13: track 0.00 -> 28.5 mm
- net GPIO27: track 0.00 -> 15.5 mm, vias 0 -> 1
- net Net-(C12-Pad1): track 0.00 -> 6.25 mm
- net Net-(C13-Pad1): track 0.00 -> 5.15 mm
- net Net-(R16-Pad1): track 0.00 -> 4.99 mm
- net Net-(R17-Pad2): track 0.00 -> 4.75 mm
- net GND: vias 0 -> 6
Other:
- net class Default: clearance 0.154 -> 0.127
- rule trace_clearance: 0.154 -> 0.127
Changed lines of the file:
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@@
     (thickness 1.6)
     (drawings 9)
-    (tracks 129)
+    (tracks 169)
     (zones 0)
     (modules 45)
@@
   )
   (setup
-    (last_trace_width 0.381)
+    (last_trace_width 0.1524)
     (user_trace_width 0.254)
     (user_trace_width 0.381)
-    (trace_clearance 0.154)
+    (trace_clearance 0.127)
     (zone_clearance 0.154)
     (zone_45_only no)
@@
   (net 89 GND)
   (net_class Default "This is the default net class."
-    (clearance 0.154)
+    (clearance 0.127)
     (trace_width 0.1524)
     (via_dia 0.508)
@@
   )
   (module Resistor_SMD:R_0402_1005Metric (layer F.Cu)
-    (at 45.72 39.878)
+    (at 45.72 39.878 180)
     (descr "Resistor SMD 0402 (1005 Metric), square (rectangular) end terminal, IPC_7351 nominal, (Body size source: IPC-SM-782 page 72, https://www.pcb-3d.com/wordpress/wp-content/uploads/ipc-sm-782a_amendment_1_and_2.pdf), generated with kicad-footprint-generator")
     (tags resistor)
@@
       (effects (font (size 0.26 0.26) (thickness 0.04)))
     )
-    (pad 2 smd roundrect (at 0.51 0) (size 0.54 0.64) (layers F.Cu F.Paste F.Mask) (roundrect_rratio 0.25)
+    (pad 2 smd roundrect (at 0.51 0 180) (size 0.54 0.64) (layers F.Cu F.Paste F.Mask) (roundrect_rratio 0.25)
       (net 39 "Net-(R3-Pad2)"))
-    (pad 1 smd roundrect (at -0.51 0) (size 0.54 0.64) (layers F.Cu F.Paste F.Mask) (roundrect_rratio 0.25)
+    (pad 1 smd roundrect (at -0.51 0 180) (size 0.54 0.64) (layers F.Cu F.Paste F.Mask) (roundrect_rratio 0.25)
       (net 40 CP_Tx))
     (model ${KISYS3DMOD}/Resistor_SMD.3dshapes/R_0402_1005Metric.wrl
@@
   (segment (start 68.798 34.818) (end 68.798 35.208) (width 0.25) (layer F.Cu) (net 1))
   (segment (start 41.232 33.34) (end 43.752 33.34) (width 0.381) (layer F.Cu) (net 2))
-  (segment (start 46.64 33.968) (end 50.927 33.968) (width 0.1524) (layer F.Cu) (net 2))
-  (segment (start 46.2 33.528) (end 46.64 33.968) (width 0.1524) (layer F.Cu) (net 2))
   (segment (start 46.2 33.683) (end 46.2 33.528) (width 0.1524) (layer F.Cu) (net 2))
   (segment (start 45.21 34.673) (end 46.2 33.683) (width 0.1524) (layer F.Cu) (net 2))
@@
   (segment (start 41.232 32.85) (end 39.751 31.369) (width 0.254) (layer F.Cu) (net 2))
   (segment (start 41.232 33.34) (end 41.232 32.85) (width 0.254) (layer F.Cu) (net 2))
+  (segment (start 48.582 33.968) (end 50.927 33.968) (width 0.1524) (layer F.Cu) (net 2))
+  (segment (start 48.142 33.528) (end 48.582 33.968) (width 0.1524) (layer F.Cu) (net 2))
+  (segment (start 46.2 33.528) (end 48.142 33.528) (width 0.1524) (layer F.Cu) (net 2))
   (segment (start 66.07 32.484) (end 66.04 32.514) (width 0.25) (layer F.Cu) (net 3))
   (segment (start 67.31 32.484) (end 66.07 32.484) (width 0.1524) (layer F.Cu) (net 3))
@@
   (segment (start 64.77 33.274) (end 65.298 33.802) (width 0.1524) (layer F.Cu) (net 3))
   (segment (start 64.77 32.514) (end 64.77 33.274) (width 0.1524) (layer F.Cu) (net 3))
+  (segment (start 46.77 36.768) (end 50.927 36.768) (width 0.1524) (layer F.Cu) (net 6))
+  (segment (start 46.2 37.338) (end 46.77 36.768) (width 0.1524) (layer F.Cu) (net 6))
+  (segment (start 46.23 37.368) (end 46.2 37.338) (width 0.1524) (layer F.Cu) (net 6))
+  (segment (start 46.23 38.608) (end 46.23 37.368) (width 0.1524) (layer F.Cu) (net 6))
+  (segment (start 47.498 32.258) (end 46.2 32.258) (width 0.1524) (layer F.Cu) (net 7))
+  (segment (start 48.508 33.268) (end 47.498 32.258) (width 0.1524) (layer F.Cu) (net 7))
+  (segment (start 50.927 33.268) (end 48.508 33.268) (width 0.1524) (layer F.Cu) (net 7))
   (segment (start 40.771 30.988) (end 41.933 30.988) (width 0.1524) (layer F.Cu) (net 8))
+  (via (at 43.688 30.988) (size 0.508) (drill 0.254) (layers F.Cu B.Cu) (net 9))
+  (segment (start 42.903 30.988) (end 43.688 30.988) (width 0.1524) (layer F.Cu) (net 9))
+  (segment (start 45.466 44.196) (end 45.466 44.958) (width 0.1524) (layer B.Cu) (net 9))
+  (segment (start 43.688 42.418) (end 45.466 44.196) (width 0.1524) (layer B.Cu) (net 9))
+  (segment (start 43.688 30.988) (end 43.688 42.418) (width 0.1524) (layer B.Cu) (net 9))
   (segment (start 40.769 29.718) (end 41.933 29.718) (width 0.1524) (layer F.Cu) (net 10))
+  (segment (start 38.84 27.574) (end 42.44 27.574) (width 0.1524) (layer F.Cu) (net 11))
+  (segment (start 64.008 26.162) (end 64.516 26.67) (width 0.1524) (layer F.Cu) (net 11))
+  (segment (start 44.845731 26.162) (end 64.008 26.162) (width 0.1524) (layer F.Cu) (net 11))
+  (segment (start 64.516 26.67) (end 64.516 28.829) (width 0.1524) (layer F.Cu) (net 11))
+  (segment (start 43.433731 27.574) (end 44.845731 26.162) (width 0.1524) (layer F.Cu) (net 11))
+  (segment (start 66.04 30.353) (end 66.04 31.494) (width 0.1524) (layer F.Cu) (net 11))
+  (segment (start 64.516 28.829) (end 66.04 30.353) (width 0.1524) (layer F.Cu) (net 11))
+  (segment (start 42.44 27.574) (end 43.433731 27.574) (width 0.1524) (layer F.Cu) (net 11))
   (segment (start 33.001 33.618) (end 32.837 33.782) (width 0.25) (layer F.Cu) (net 12))
   (segment (start 30.988 34.798) (end 30.988 37.375) (width 0.25) (layer F.Cu) (net 12))
@@
   (segment (start 34.553 33.618) (end 35.433 32.738) (width 0.381) (layer F.Cu) (net 12))
   (segment (start 33.001 33.618) (end 34.553 33.618) (width 0.381) (layer F.Cu) (net 12))
-  (segment (start 49.332 32.568) (end 47.8155 31.0515) (width 0.254) (layer F.Cu) (net 12))
-  (segment (start 47.8155 29.5275) (end 47.8155 31.0515) (width 0.254) (layer B.Cu) (net 12))
-  (segment (start 45.466 27.178) (end 47.8155 29.5275) (width 0.254) (layer B.Cu) (net 12))
-  (segment (start 50.927 32.568) (end 49.332 32.568) (width 0.254) (layer F.Cu) (net 12))
-  (via (at 47.8155 31.0515) (size 0.508) (drill 0.254) (layers F.Cu B.Cu) (net 12))
   (via (at 37.084 32.766) (size 0.508) (drill 0.254) (layers F.Cu B.Cu) (net 12))
   (segment (start 37.056 32.738) (end 37.084 32.766) (width 0.381) (layer F.Cu) (net 12))
@@
   (segment (start 37.658 33.34) (end 39.032 33.34) (width 0.381) (layer F.Cu) (net 12))
   (segment (start 37.084 32.766) (end 37.658 33.34) (width 0.381) (layer F.Cu) (net 12))
+  (via (at 47.878999 31.75) (size 0.508) (drill 0.254) (layers F.Cu B.Cu) (net 12))
+  (segment (start 50.927 32.568) (end 48.696999 32.568) (width 0.254) (layer F.Cu) (net 12))
+  (segment (start 48.696999 32.568) (end 47.878999 31.75) (width 0.254) (layer F.Cu) (net 12))
+  (segment (start 45.466 27.178) (end 47.878999 29.590999) (width 0.254) (layer B.Cu) (net 12))
+  (segment (start 47.878999 29.590999) (end 47.878999 31.75) (width 0.254) (layer B.Cu) (net 12))
+  (segment (start 35.582 27.574) (end 31.982 27.574) (width 0.1524) (layer F.Cu) (net 24))
+  (segment (start 36.703 46.101) (end 37.846 44.958) (width 0.1524) (layer F.Cu) (net 24))
+  (segment (start 34.544 46.101) (end 36.703 46.101) (width 0.1524) (layer F.Cu) (net 24))
+  (segment (start 34.036 44.323) (end 34.036 45.593) (width 0.1524) (layer F.Cu) (net 24))
+  (segment (start 30.099 40.386) (end 34.036 44.323) (width 0.1524) (layer F.Cu) (net 24))
+  (segment (start 34.036 45.593) (end 34.544 46.101) (width 0.1524) (layer F.Cu) (net 24))
+  (segment (start 30.099 29.457) (end 30.099 40.386) (width 0.1524) (layer F.Cu) (net 24))
+  (segment (start 31.982 27.574) (end 30.099 29.457) (width 0.1524) (layer F.Cu) (net 24))
   (segment (start 36.943 38.878) (end 37.682 38.878) (width 0.1524) (layer F.Cu) (net 38))
   (segment (start 35.433 40.388) (end 36.943 38.878) (width 0.1524) (layer F.Cu) (net 38))
@@
   (segment (start 34.943 34.818) (end 35.433 35.308) (width 0.1524) (layer F.Cu) (net 46))
   (segment (start 33.001 34.818) (end 34.943 34.818) (width 0.1524) (layer F.Cu) (net 46))
+  (segment (start 46.93 35.368) (end 50.927 35.368) (width 0.1524) (layer F.Cu) (net 47))
+  (segment (start 46.23 36.068) (end 46.93 35.368) (width 0.1524) (layer F.Cu) (net 47))
+  (segment (start 49.527 34.668) (end 50.927 34.668) (width 0.1524) (layer F.Cu) (net 48))
+  (segment (start 46.36 34.668) (end 49.527 34.668) (width 0.1524) (layer F.Cu) (net 48))
+  (segment (start 46.23 34.798) (end 46.36 34.668) (width 0.1524) (layer F.Cu) (net 48))
   (segment (start 32.004 35.4376) (end 32.004 36.1984) (width 0.1524) (layer F.Cu) (net 66))
   (segment (start 32.1236 36.318) (end 33.001 36.318) (width 0.1524) (layer F.Cu) (net 66))
@@
   (segment (start 39.243 37.211) (end 39.37 37.211) (width 0.1524) (layer B.Cu) (net 67))
   (segment (start 40.132 36.449) (end 40.132 37.428) (width 0.1524) (layer F.Cu) (net 67))
+  (via (at 44.577 37.338) (size 0.508) (drill 0.254) (layers F.Cu B.Cu) (net 89))
+  (via (at 44.577 36.068) (size 0.508) (drill 0.254) (layers F.Cu B.Cu) (net 89))
+  (via (at 35.433 30.734) (size 0.508) (drill 0.254) (layers F.Cu B.Cu) (net 89))
+  (via (at 37.084 34.29) (size 0.508) (drill 0.254) (layers F.Cu B.Cu) (net 89))
+  (via (at 33.782 26.289) (size 0.508) (drill 0.254) (layers F.Cu B.Cu) (net 89))
+  (via (at 40.64 26.289) (size 0.508) (drill 0.254) (layers F.Cu B.Cu) (net 89))
   (zone (net 89) (net_name GND) (layer F.Cu) (hatch edge 0.508)
     (connect_pads yes (clearance 0.154))

Commit message: .
Parts:
- moved C2 5.07 mm to (42.8, 32.9), turned to 270 degrees
- moved D1 4.76 mm to (37.7, 30.2), turned to 0 degrees
- moved C1 4.58 mm to (41.4, 32.9), turned to 270 degrees
- moved C8 4.03 mm to (53.9, 35.1)
- moved R14 2.39 mm to (63.9, 31.0)
- moved C6 2.07 mm to (53.9, 33.1)
- moved C10 2.07 mm to (53.9, 31.1)
- moved R12 1.97 mm to (42.2, 30.2)
- moved C7 1.85 mm to (65.5, 31.5), turned to 0 degrees
- moved D2 1.85 mm to (44.2, 30.2)
- moved U2 1.73 mm to (38.7, 33.3)
- moved R6 1.70 mm to (65.5, 30.5), turned to 0 degrees
- moved C9 1.27 mm to (62.7, 31.0)
- moved U1 1.02 mm to (40.1, 38.9)
- moved C4 0.92 mm to (58.3, 40.1)
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Routing:
- net +3V3: track 32.0 -> 102.1 mm, vias 0 -> 9
- net GPIO27: track 15.5 -> 58.7 mm, vias 1 -> 0
- net GPIO22: track 0.00 -> 35.8 mm, vias 0 -> 2
- net GPIO5: track 0.00 -> 34.3 mm, vias 0 -> 1
- net GPIO2: track 0.00 -> 32.8 mm, vias 0 -> 1
- net GPIO4: track 0.00 -> 32.2 mm, vias 0 -> 1
- net CP_Rx: track 0.00 -> 32.2 mm, vias 0 -> 3
- net GPIO0: track 0.00 -> 29.6 mm, vias 0 -> 2
- net GPIO13: track 28.5 -> 57.4 mm, vias 0 -> 1
- net CP_Tx: track 0.00 -> 28.8 mm, vias 0 -> 2
- net GPIO14: track 0.00 -> 27.1 mm, vias 0 -> 1
- net EN: track 5.47 -> 32.4 mm, vias 0 -> 5
- net GPIO21: track 0.00 -> 26.8 mm, vias 0 -> 2
- net RTS: track 0.00 -> 23.9 mm, vias 0 -> 2
- net GPIO12: track 0.00 -> 23.3 mm, vias 0 -> 3
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- removed copper zone on F.Cu, net (none)
