File: esp32-nano.kicad_pcb (KiCad board)
At the start: 2 copper layers, 52.8 x 21.3 mm, 45 parts, among them K1 SW_MEC_5E, K2 SW_MEC_5E, P2 Conn_01x12, P3 Conn_01x18, U1 CP2102N-A01-GQFN28, U2 ME6211C33M5G, U3 MPU-6050, U4 ESP32PICO_D4, U5 OLED-12880

Commit message: .
Parts:
- added G***: LOGO, logo:logo, B.Cu at (59.3, 36.5)
Routing:
- net +3V3: track 102.1 -> 100.9 mm
- net GND: vias 74 -> 89
Other:
- board text added: "0"
- board text added: "10"
- board text added: "11"
- board text added: "12"
- board text added: "13"
- board text added: "14"
- board text added: "15"
- board text added: "18"
- board text added: "19"
- board text added: "2"
- board text added: "23"
- board text added: "25"
- board text added: "26"
- board text added: "27"
- board text added: "34"
- board text added: "35"
- board text added: "36"
- board text added: "37"
- board text added: "38"
- board text added: "39"
- board text added: "3V3"
- board text added: "4"
- board text added: "5"
- board text added: "6"
- board text added: "7"
- board text added: "8"
- board text added: "9"
- board text added: "BTN"
- board text added: "GND"
- board text added: "RST"
- board text added: "VBUS"
