File: esp32-nano.sch (KiCad schematic (older format))
At the start: 14 parts, among them U1 CP2102N-A01-GQFN28, U2 ME6211C33M5G

Commit message: .
Parts:
- added A1: Antenna, CA-C03:CA-C03, symbol Device:Antenna
- added C12, C13, C4: 10uF, Capacitor_SMD:C_0402_1005Metric, symbol Device:C
- added C5: 0.1uF, Capacitor_SMD:C_0402_1005Metric, symbol Device:C
- added D1: ORANGE, LED_SMD:LED_0402_1005Metric, symbol Device:LED
- added D2: GREEN, LED_SMD:LED_0402_1005Metric, symbol Device:LED
- added K1, K2: SW_MEC_5E, SKSCLCE010:SKSCLCE010, symbol Switch:SW_MEC_5E
- added P2: Conn_01x12, symbol Connector_Generic:Conn_01x12
- added P3: Conn_01x18, symbol Connector_Generic:Conn_01x18
- added R12, R13, R9: 10K, Resistor_SMD:R_0402_1005Metric, symbol Device:R
- added R14: 1K, Resistor_SMD:R_0402_1005Metric, symbol Device:R
- added R16: 560K, Resistor_SMD:R_0402_1005Metric, symbol Device:R
- added R17: 4.7K, Resistor_SMD:R_0402_1005Metric, symbol Device:R
- added U4: ESP32PICO_D4, ESP32_PICO_D4:ESP32_PICO_D4, symbol esp32pico_d4:ESP32PICO_D4
- added U5: OLED-12880, OLED-12880:OLED-12880, symbol OLED-12880:OLED-12880
- C1, C14, C2: footprint (none) -> Capacitor_SMD:C_0402_1005Metric
- R1, R3, R4, R5, R7, R8: footprint (none) -> Resistor_SMD:R_0402_1005Metric
Connections:
- net labels added: FLASH_CLK, FLASH_CS, FLASH_SD0, FLASH_SD1, FLASH_SD2, FLASH_SD3, GPIO10, GPIO12, GPIO13, GPIO14, GPIO15, GPIO18, GPIO19, GPIO2, GPIO21, GPIO22, GPIO23, GPIO25, GPIO26, GPIO27, GPIO32, GPIO33, GPIO34, GPIO35, GPIO37, GPIO38, GPIO4, GPIO5, GPIO9, SENSOR_VN, SENSOR_VP
- wire segments 61 -> 164
Other:
- moved on the sheet: C1, C14, C2, R1, R3, R4, R5, R7, R8, U1, U2, USB1

Commit message: .
Parts:
- added C10, C7, C8: 0.1uF, Capacitor_SMD:C_0402_1005Metric, symbol Device:C
- added C6: 10nF, Capacitor_SMD:C_0402_1005Metric, symbol Device:C
- added C9: 2.2nF, Capacitor_SMD:C_0402_1005Metric, symbol Device:C
- added R6: 10K, Resistor_SMD:R_0402_1005Metric, symbol Device:R
- added U3: MPU-6050, Sensor_Motion:InvenSense_QFN-24_4x4mm_P0.5mm, symbol Sensor_Motion:MPU-6050
- P2: footprint (none) -> 12pin:12pin
- P3: footprint (none) -> 18pin:18pin
- U2: footprint ME6211C33M5G:SOT95P282X145-5N -> Package_TO_SOT_SMD:SOT-23-5
- VT1, VT2: footprint Package_TO_SOT_THT:TO-92_Inline -> Package_TO_SOT_SMD:SOT-23; symbol Transistor_BJT:S8050 -> S8050:S8050
Connections:
- net labels added: GPIO11, GPIO6, GPIO7, GPIO8
- net labels removed: FLASH_CLK, FLASH_SD1, FLASH_SD2, FLASH_SD3
- wire segments 164 -> 186
Other:
- moved on the sheet: C12, C13, R13, R16, R17, R4, R5, U5

Commit message: .
Parts:
- added C11: 10uF, Capacitor_SMD:C_0402_1005Metric, symbol Device:C
Connections:
- net +3V3: now also C11.2
- net GND: now also C11.1; no longer K2.3 (K), K2.4 (A)
- net GPIO13: now also K2.3 (K), K2.4 (A)
Changed lines of the file:
@@
 Wire Wire Line
 	1250 7300 1400 7300
-$Comp
-L power:GND #PWR0138
-U 1 1 617DCFBC
-P 2000 7300
-F 0 "#PWR0138" H 2000 7050 50  0001 C CNN
-F 1 "GND" V 2005 7172 50  0000 R CNN
-F 2 "" H 2000 7300 50  0001 C CNN
-F 3 "" H 2000 7300 50  0001 C CNN
-	1    2000 7300
-	0    -1   -1   0
-$EndComp
 Wire Wire Line
 	1800 7300 2000 7300
@@
 GPIO8
 $Comp
-L power:VBUS #PWR?
+L power:VBUS #PWR0103
 U 1 1 6180D0A9
 P 950 1100
-F 0 "#PWR?" H 950 950 50  0001 C CNN
+F 0 "#PWR0103" H 950 950 50  0001 C CNN
 F 1 "VBUS" V 965 1227 50  0000 L CNN
 F 2 "" H 950 1100 50  0001 C CNN
@@
 	0    -1   -1   0
 $EndComp
+Text GLabel 2000 7300 2    50   Input ~ 0
+GPIO13
+$Comp
+L power:GND #PWR0138
+U 1 1 61603AC9
+P 6050 4300
+F 0 "#PWR0138" H 6050 4050 50  0001 C CNN
+F 1 "GND" V 6055 4172 50  0000 R CNN
+F 2 "" H 6050 4300 50  0001 C CNN
+F 3 "" H 6050 4300 50  0001 C CNN
+	1    6050 4300
+	0    -1   -1   0
+$EndComp
+$Comp
+L Device:C C11
+U 1 1 61604B51
+P 5850 4300
+F 0 "C11" V 5598 4300 50  0000 C CNN
+F 1 "10uF" V 5689 4300 50  0000 C CNN
+F 2 "Capacitor_SMD:C_0402_1005Metric" H 5888 4150 50  0001 C CNN
+F 3 "~" H 5850 4300 50  0001 C CNN
+	1    5850 4300
+	0    1    1    0
+$EndComp
+$Comp
+L power:+3V3 #PWR0148
+U 1 1 61602827
+P 5650 4300
+F 0 "#PWR0148" H 5650 4150 50  0001 C CNN
+F 1 "+3V3" V 5665 4428 50  0000 L CNN
+F 2 "" H 5650 4300 50  0001 C CNN
+F 3 "" H 5650 4300 50  0001 C CNN
+	1    5650 4300
+	0    -1   -1   0
+$EndComp
+Wire Wire Line
+	5650 4300 5700 4300
+Wire Wire Line
+	6000 4300 6050 4300
 $EndSCHEMATC

Commit message: .
Parts:
- A1: footprint CA-C03:CA-C03 -> Antenna:CA-C03
- K1, K2: footprint SKSCLCE010:SKSCLCE010 -> Button:SKSC_NO_HOLE
- P2: footprint 12pin:12pin -> Connector_Custom:PinHeader_1x12_P2.54mm
- P3: footprint 18pin:18pin -> Connector_Custom:PinHeader_1x18_P2.54mm
- U2: symbol ME6211C33M5G:ME6211C33M5G -> LDO:ME6211C33M5G-N; Max Output Current (none) -> 800mA
- U4: footprint ESP32_PICO_D4:ESP32_PICO_D4 -> SOC:ESP32_PICO_D4; symbol esp32pico_d4:ESP32PICO_D4 -> SOC:ESP32PICO_D4
- USB1: symbol USB_C_16_PIN:USB_C_16_PIN -> Connector_Custom:USB_C_16_PIN
- VT1, VT2: symbol S8050:S8050 -> Triode:S8050
Other:
- moved on the sheet: C1, C2, U2
Changed lines of the file:
@@
 L power:GND #PWR0102
 U 1 1 615115B7
-P 950 1000
-F 0 "#PWR0102" H 950 750 50  0001 C CNN
-F 1 "GND" V 955 872 50  0000 R CNN
-F 2 "" H 950 1000 50  0001 C CNN
-F 3 "" H 950 1000 50  0001 C CNN
-	1    950  1000
-	0    1    1    0
+P 1750 1450
+F 0 "#PWR0102" H 1750 1200 50  0001 C CNN
+F 1 "GND" V 1755 1322 50  0000 R CNN
+F 2 "" H 1750 1450 50  0001 C CNN
+F 3 "" H 1750 1450 50  0001 C CNN
+	1    1750 1450
+	1    0    0    -1
 $EndComp
 $Comp
@@
 L power:+3V3 #PWR0105
 U 1 1 61514C03
-P 2950 1000
-F 0 "#PWR0105" H 2950 850 50  0001 C CNN
-F 1 "+3V3" V 2965 1128 50  0000 L CNN
-F 2 "" H 2950 1000 50  0001 C CNN
-F 3 "" H 2950 1000 50  0001 C CNN
-	1    2950 1000
+P 2900 900
+F 0 "#PWR0105" H 2900 750 50  0001 C CNN
+F 1 "+3V3" V 2915 1028 50  0000 L CNN
+F 2 "" H 2900 900 50  0001 C CNN
+F 3 "" H 2900 900 50  0001 C CNN
+	1    2900 900
 	0    1    1    0
 $EndComp
@@
 L power:GND #PWR0106
 U 1 1 6151566A
-P 2400 1400
-F 0 "#PWR0106" H 2400 1150 50  0001 C CNN
-F 1 "GND" H 2405 1227 50  0000 C CNN
-F 2 "" H 2400 1400 50  0001 C CNN
-F 3 "" H 2400 1400 50  0001 C CNN
-	1    2400 1400
+P 2350 1300
+F 0 "#PWR0106" H 2350 1050 50  0001 C CNN
+F 1 "GND" H 2355 1127 50  0000 C CNN
+F 2 "" H 2350 1300 50  0001 C CNN
+F 3 "" H 2350 1300 50  0001 C CNN
+	1    2350 1300
 	1    0    0    -1
 $EndComp
@@
 L Device:C C1
 U 1 1 615163AF
-P 2400 1200
-F 0 "C1" H 2515 1246 50  0000 L CNN
-F 1 "1uF" H 2515 1155 50  0000 L CNN
-F 2 "Capacitor_SMD:C_0402_1005Metric" H 2438 1050 50  0001 C CNN
-F 3 "~" H 2400 1200 50  0001 C CNN
-	1    2400 1200
+P 2350 1100
+F 0 "C1" H 2465 1146 50  0000 L CNN
+F 1 "1uF" H 2465 1055 50  0000 L CNN
+F 2 "Capacitor_SMD:C_0402_1005Metric" H 2388 950 50  0001 C CNN
+F 3 "~" H 2350 1100 50  0001 C CNN
+	1    2350 1100
 	1    0    0    -1
 $EndComp
@@
 L Device:C C2
 U 1 1 615175EE
-P 2800 1200
-F 0 "C2" H 2915 1246 50  0000 L CNN
-F 1 "10uF" H 2915 1155 50  0000 L CNN
-F 2 "Capacitor_SMD:C_0402_1005Metric" H 2838 1050 50  0001 C CNN
-F 3 "~" H 2800 1200 50  0001 C CNN
-	1    2800 1200
+P 2750 1100
+F 0 "C2" H 2865 1146 50  0000 L CNN
+F 1 "10uF" H 2865 1055 50  0000 L CNN
+F 2 "Capacitor_SMD:C_0402_1005Metric" H 2788 950 50  0001 C CNN
+F 3 "~" H 2750 1100 50  0001 C CNN
+	1    2750 1100
 	1    0    0    -1
 $EndComp
@@
 L power:GND #PWR0107
 U 1 1 615180AE
-P 2800 1400
-F 0 "#PWR0107" H 2800 1150 50  0001 C CNN
-F 1 "GND" H 2805 1227 50  0000 C CNN
-F 2 "" H 2800 1400 50  0001 C CNN
-F 3 "" H 2800 1400 50  0001 C CNN
-	1    2800 1400
+P 2750 1300
+F 0 "#PWR0107" H 2750 1050 50  0001 C CNN
+F 1 "GND" H 2755 1127 50  0000 C CNN
+F 2 "" H 2750 1300 50  0001 C CNN
+F 3 "" H 2750 1300 50  0001 C CNN
+	1    2750 1300
 	1    0    0    -1
 $EndComp
@@
 $EndComp
 $Comp
-L S8050:S8050 VT1
+L Triode:S8050 VT1
 U 1 1 61525401
 P 1700 2200
@@
 RTS
 Wire Wire Line
-	1200 1100 1050 1100
+	1400 1100 1050 1100
 Wire Wire Line
 	1050 1100 1050 1150
@@
 	1050 1100 950  1100
 Wire Wire Line
-	2400 1000 2400 1050
-Connection ~ 2400 1000
-Wire Wire Line
-	2400 1350 2400 1400
-Wire Wire Line
-	2400 1000 2800 1000
-Wire Wire Line
-	2800 1050 2800 1000
-Connection ~ 2800 1000
-Wire Wire Line
-	2800 1000 2950 1000
-Wire Wire Line
-	2800 1350 2800 1400
+	2350 900  2350 950
+Connection ~ 2350 900
+Wire Wire Line
+	2350 1250 2350 1300
+Wire Wire Line
+	2350 900  2750 900
+Wire Wire Line
+	2750 950  2750 900
+Connection ~ 2750 900
+Wire Wire Line
+	2750 900  2900 900
+Wire Wire Line
+	2750 1250 2750 1300
 Wire Wire Line
 	4350 1600 4100 1600
@@
 	1600 2000 1350 2000
 $Comp
-L USB_C_16_PIN:USB_C_16_PIN USB1
+L Connector_Custom:USB_C_16_PIN USB1
 U 1 1 61553A6A
 P 2250 4150
@@
 	2800 4400 2950 4400
 Wire Wire Line
-	2300 1000 2400 1000
-$Comp
-L ME6211C33M5G:ME6211C33M5G U2
+	2100 900  2350 900
+$Comp
+L LDO:ME6211C33M5G-N U2
 U 1 1 6150E1CB
-P 1200 900
-F 0 "U2" H 1750 1165 50  0000 C CNN
-F 1 "ME6211C33M5G" H 1750 1074 50  0000 C CNN
-F 2 "Package_TO_SOT_SMD:SOT-23-5" H 1400 450 50  0001 L CNN
-F 3 "http://xinhuidianzi.com.cn/UploadSysFiles/files/LDO-series/ME6211-Series_E15.0.pdf" H 1400 350 50  0001 L CNN
-F 4 "High Speed LDO Regulators, High PSRR, Low noise, ME6211 Series" H 1400 250 50  0001 L CNN "Description"
-F 5 "1.45" H 1400 150 50  0001 L CNN "Height"
-F 6 "Microne" H 1400 50  50  0001 L CNN "Manufacturer_Name"
-F 7 "ME6211C33M5G" H 1400 -50 50  0001 L CNN "Manufacturer_Part_Number"
-F 8 "" H 2150 400 50  0001 L CNN "Mouser Part Number"
-F 9 "" H 2150 300 50  0001 L CNN "Mouser Price/Stock"
-F 10 "" H 2150 200 50  0001 L CNN "Arrow Part Number"
-F 11 "" H 2150 100 50  0001 L CNN "Arrow Price/Stock"
-	1    1200 900
-	1    0    0    -1
-$EndComp
-$Comp
-L esp32pico_d4:ESP32PICO_D4 U4
+P 1750 1000
+F 0 "U2" H 1550 1350 50  0000 C CNN
+F 1 "ME6211C33M5G" H 1800 1250 50  0000 C CNN
+F 2 "Package_TO_SOT_SMD:SOT-23-5" H 1950 550 50  0001 L CNN
+F 3 "http://xinhuidianzi.com.cn/UploadSysFiles/files/LDO-series/ME6211-Series_E15.0.pdf" H 1950 450 50  0001 L CNN
+F 4 "High Speed LDO Regulators, High PSRR, Low noise, ME6211 Series" H 1950 350 50  0001 L CNN "Description"
+F 5 "1.45" H 1950 250 50  0001 L CNN "Height"
+F 6 "Microne" H 1950 150 50  0001 L CNN "Manufacturer_Name"
+F 7 "ME6211C33M5G" H 1950 50  50  0001 L CNN "Manufacturer_Part_Number"
+F 8 "" H 2700 500 50  0001 L CNN "Mouser Part Number"
+F 9 "" H 2700 400 50  0001 L CNN "Mouser Price/Stock"
+F 10 "" H 2700 300 50  0001 L CNN "Arrow Part Number"
+F 11 "" H 2700 200 50  0001 L CNN "Arrow Price/Stock"
+F 12 "800mA" H 1750 1000 50  0001 C CNN "Max Output Current"
+	1    1750 1000
+	1    0    0    -1
+$EndComp
+$Comp
+L SOC:ESP32PICO_D4 U4
 U 1 1 61533328
 P 8300 3350
 F 0 "U4" H 8300 3300 60  0000 L CNN
 F 1 "ESP32PICO_D4" H 9850 3300 60  0000 L CNN
-F 2 "ESP32_PICO_D4:ESP32_PICO_D4" H 8300 3350 60  0001 C CNN
+F 2 "SOC:ESP32_PICO_D4" H 8300 3350 60  0001 C CNN
 F 3 "" H 8300 3350 60  0001 C CNN
 	1    8300 3350
@@
 F 0 "A1" H 7680 1689 50  0000 L CNN
 F 1 "Antenna" H 7680 1598 50  0000 L CNN
-F 2 "CA-C03:CA-C03" H 7600 1700 50  0001 C CNN
+F 2 "Antenna:CA-C03" H 7600 1700 50  0001 C CNN
 F 3 "~" H 7600 1700 50  0001 C CNN
 	1    7600 1700
@@
 F 0 "P2" H 7318 4325 50  0000 C CNN
 F 1 "Conn_01x12" H 7318 4416 50  0000 C CNN
-F 2 "12pin:12pin" H 7400 5150 50  0001 C CNN
+F 2 "Connector_Custom:PinHeader_1x12_P2.54mm" H 7400 5150 50  0001 C CNN
 F 3 "~" H 7400 5150 50  0001 C CNN
 	1    7400 5150
@@
 F 0 "P3" H 8918 4325 50  0000 C CNN
 F 1 "Conn_01x18" H 8918 4416 50  0000 C CNN
-F 2 "18pin:18pin" H 9000 5450 50  0001 C CNN
+F 2 "Connector_Custom:PinHeader_1x18_P2.54mm" H 9000 5450 50  0001 C CNN
 F 3 "~" H 9000 5450 50  0001 C CNN
 	1    9000 5450
@@
 F 0 "K1" H 1600 7085 50  0000 C CNN
 F 1 "SW_MEC_5E" H 1600 6994 50  0000 C CNN
-F 2 "SKSCLCE010:SKSCLCE010" H 1600 7000 50  0001 C CNN
+F 2 "Button:SKSC_NO_HOLE" H 1600 7000 50  0001 C CNN
 F 3 "http://www.apem.com/int/index.php?controller=attachment&id_attachment=1371" H 1600 7000 50  0001 C CNN
 	1    1600 6700
@@
 F 0 "K2" H 1600 7785 50  0000 C CNN
 F 1 "SW_MEC_5E" H 1600 7694 50  0000 C CNN
-F 2 "SKSCLCE010:SKSCLCE010" H 1600 7700 50  0001 C CNN
+F 2 "Button:SKSC_NO_HOLE" H 1600 7700 50  0001 C CNN
 F 3 "http://www.apem.com/int/index.php?controller=attachment&id_attachment=1371" H 1600 7700 50  0001 C CNN
 	1    1600 7400
@@
 $EndComp
 Wire Wire Line
-	1200 900  1000 900
+	1400 900  1000 900
 Wire Wire Line
 	1000 900  950  900
 Connection ~ 1000 900
-Wire Wire Line
-	950  1000 1200 1000
-$Comp
-L S8050:S8050 VT2
+$Comp
+L Triode:S8050 VT2
 U 1 1 61527A63
 P 1700 2950
@@
 Wire Wire Line
 	6000 4300 6050 4300
+Wire Wire Line
+	1750 1300 1750 1450
 $EndSCHEMATC

Commit message: .
Connections:
- net FLASH_CS: no longer names the net of U4.25 (IO16)
- net FLASH_SD0: no longer names the net of U4.27 (IO17)
- no-connect marks 0 -> 31
Changed lines of the file:
@@
-	1    0    0    -1
-$EndComp
-$Comp
-L Interface_USB:CP2102N-A01-GQFN28 U1
-U 1 1 61518730
-P 4850 2200
-F 0 "U1" H 4850 811 50  0000 C CNN
-F 1 "CP2102N-A01-GQFN28" H 4850 720 50  0000 C CNN
-F 2 "Package_DFN_QFN:QFN-28-1EP_5x5mm_P0.5mm_EP3.35x3.35mm" H 5300 1000 50  0001 L CNN
-F 3 "https://www.silabs.com/documents/public/data-sheets/cp2102n-datasheet.pdf" H 4900 1450 50  0001 C CNN
-	1    4850 2200
 	1    0    0    -1
 $EndComp
@@
 Wire Wire Line
 	2650 4600 2800 4600
-Connection ~ 2800 4400
-Wire Wire Line
-	2800 4400 2950 4400
 Wire Wire Line
 	2100 900  2350 900
@@
 Text GLabel 10350 2800 2    50   Input ~ 0
 GPIO9
-Text GLabel 10350 2900 2    50   Input ~ 0
-FLASH_SD0
-Text GLabel 10350 3100 2    50   Input ~ 0
-FLASH_CS
 Wire Wire Line
 	10200 2000 10350 2000
@@
 Wire Wire Line
 	10200 2800 10350 2800
-Wire Wire Line
-	10200 2900 10350 2900
-Wire Wire Line
-	10200 3100 10350 3100
 Text GLabel 9250 1400 1    50   Input ~ 0
 GPIO21
@@
 	6000 4300 6050 4300
 Wire Wire Line
-	1750 1300 1750 1450
+	1750 1300 1750 1400
+NoConn ~ 5350 1100
+NoConn ~ 5350 1500
+NoConn ~ 4850 900
+NoConn ~ 5350 1700
+NoConn ~ 5350 1800
+NoConn ~ 5350 2000
+NoConn ~ 5350 2100
+NoConn ~ 5350 2300
+NoConn ~ 5350 2400
+NoConn ~ 5350 2500
+NoConn ~ 5350 2700
+NoConn ~ 5350 2800
+NoConn ~ 5350 2900
+NoConn ~ 5350 3000
+NoConn ~ 5350 3100
+NoConn ~ 5350 3200
+NoConn ~ 5350 3300
+NoConn ~ 2650 3900
+NoConn ~ 1850 4200
+NoConn ~ 5100 6800
+NoConn ~ 5100 6700
+NoConn ~ 5100 6500
+NoConn ~ 4900 5450
+NoConn ~ 10200 3000
+NoConn ~ 8650 1550
+NoConn ~ 8750 1550
+NoConn ~ 8950 1550
+NoConn ~ 9050 1550
+NoConn ~ 4900 4250
+Connection ~ 2800 4400
+Wire Wire Line
+	2800 4400 2950 4400
+$Comp
+L Interface_USB:CP2102N-A01-GQFN28 U1
+U 1 1 61518730
+P 4850 2200
+F 0 "U1" H 4850 811 50  0000 C CNN
+F 1 "CP2102N-A01-GQFN28" H 4850 720 50  0000 C CNN
+F 2 "Package_DFN_QFN:QFN-28-1EP_5x5mm_P0.5mm_EP3.35x3.35mm" H 5300 1000 50  0001 L CNN
+F 3 "https://www.silabs.com/documents/public/data-sheets/cp2102n-datasheet.pdf" H 4900 1450 50  0001 C CNN
+	1    4850 2200
+	1    0    0    -1
+$EndComp
+$Comp
+L power:PWR_FLAG #GND0101
+U 1 1 618AE67A
+P 1850 1400
+F 0 "#GND0101" H 1850 1475 50  0001 C CNN
+F 1 "PWR_FLAG" H 1918 1442 50  0000 L CNN
+F 2 "" H 1850 1400 50  0001 C CNN
+F 3 "~" H 1850 1400 50  0001 C CNN
+	1    1850 1400
+	1    0    0    -1
+$EndComp
+Wire Wire Line
+	1850 1400 1750 1400
+Connection ~ 1750 1400
+Wire Wire Line
+	1750 1400 1750 1450
+NoConn ~ 10200 3100
+NoConn ~ 10200 2900
 $EndSCHEMATC

Commit message: 引出psram
Parts:
- R14: value 1K -> 0R
- R9: value 10K -> 3K
Connections:
- net GPIO9: now also U4.27 (IO17); no longer U4.28 (SD2)
- net VDD_SIO: now reaches U4.26 (VDD_SDIO_NC)
- net VDD_SIO: now also P3.16 (Pin_16)
- net GPIO4: no longer names the net of U4.24 (IO4)
- net GPIO4: no longer P3.16 (Pin_16)
- no-connect marks 31 -> 29
Changed lines of the file:
@@
 Text GLabel 9650 3650 3    50   Input ~ 0
 GPIO0
-Text GLabel 9750 3650 3    50   Input ~ 0
-GPIO4
 Wire Wire Line
 	8650 3550 8650 3650
@@
 Wire Wire Line
 	9650 3550 9650 3650
-Wire Wire Line
-	9750 3550 9750 3650
 $Comp
 L power:+3V3 #PWR0120
@@
 Text GLabel 10350 2700 2    50   Input ~ 0
 GPIO10
-Text GLabel 10350 2800 2    50   Input ~ 0
+Text GLabel 10350 2900 2    50   Input ~ 0
 GPIO9
 Wire Wire Line
@@
 Wire Wire Line
 	10200 2700 10350 2700
-Wire Wire Line
-	10200 2800 10350 2800
 Text GLabel 9250 1400 1    50   Input ~ 0
 GPIO21
@@
 P 1750 5300
 F 0 "R9" V 1650 5300 50  0000 C CNN
-F 1 "10K" V 1850 5300 50  0000 C CNN
+F 1 "3K" V 1850 5300 50  0000 C CNN
 F 2 "Resistor_SMD:R_0402_1005Metric" V 1680 5300 50  0001 C CNN
 F 3 "~" H 1750 5300 50  0001 C CNN
@@
 	9350 4550 9450 4550
 Text GLabel 9200 4750 2    50   Input ~ 0
-GPIO4
+VDD_SIO
 Text GLabel 9200 4850 2    50   Input ~ 0
 GPIO13
@@
 P 2150 6600
 F 0 "R14" V 1943 6600 50  0000 C CNN
-F 1 "1K" V 2034 6600 50  0000 C CNN
+F 1 "0R" V 2034 6600 50  0000 C CNN
 F 2 "Resistor_SMD:R_0402_1005Metric" V 2080 6600 50  0001 C CNN
 F 3 "~" H 2150 6600 50  0001 C CNN
@@
 NoConn ~ 5100 6500
 NoConn ~ 4900 5450
-NoConn ~ 10200 3000
 NoConn ~ 8650 1550
 NoConn ~ 8750 1550
@@
 	1750 1400 1750 1450
 NoConn ~ 10200 3100
-NoConn ~ 10200 2900
+Wire Wire Line
+	10200 2900 10350 2900
+Text GLabel 10350 3000 2    50   Input ~ 0
+VDD_SIO
+Wire Wire Line
+	10200 3000 10350 3000
 $EndSCHEMATC

Commit message: .
Connections:
- net GPIO9 renamed GPIO17
Changed lines of the file:
@@
 GPIO10
 Text GLabel 10350 2900 2    50   Input ~ 0
-GPIO9
+GPIO17
 Wire Wire Line
 	10200 2000 10350 2000
@@
 GPIO27
 Text GLabel 9200 5250 2    50   Input ~ 0
-GPIO9
+GPIO17
 Text GLabel 9200 5350 2    50   Input ~ 0
 GPIO10
